Commit message: Modified urdf and complete
Signed-off-by: jeonggeun Lim <jglim@DESKTOP-U1I4OU5.localdomain>

File: description/urdf/rb_amr.urdf (robot description, URDF)
Before this commit: robot rb_amr, 3 links, 2 joints
Links:
- added link base_visual; visual mesh filename=package://description/meshes/RB_AMR_ASSY.STL scale=0.001 0.001 0.001
- link base_link: mass 10.0 -> 30.0; geometry collision box size=0.40 0.30 0.20
Joints:
- added joint base_visual_joint: type fixed, parent base_link, child base_visual, origin xyz=0 0 0 rpy=0 0 -1.5708

Commit message: Added lidar
Signed-off-by: Jeonggeun Lim <jglim@inhatc.ac.kr>

File: description/urdf/rb_amr.urdf (robot description, URDF)
Before this commit: robot rb_amr, 4 links, 3 joints
Links:
- added link lidar_link, mass 0.2; visual cylinder length=0.05 radius=0.03
- link base_link: geometry collision box size=0.40 0.20 0.20
Joints:
- added joint lidar_joint: type fixed, parent base_link, child lidar_link, origin xyz=0.14 0.00 0.20 rpy=0 0 0
